File: Electrical/uC_Board/uC_board.kicad_pcb (KiCad board)
At the start: 2 copper layers, 45 x 18 mm, 27 parts, among them J1 Card Edge Connector, J2 Arduino Breakout Pins, Q1 BC850, SW1 SW_Push, U1 ATmega328PB-AU, U2 OPA2381, U3 LM1117MPX-5.0, X1 CSTNE16M0V530000R0

Commit message: Finalized Housing.
Routing:
- net GND: track 85.8 -> 83.4 mm
Changed lines of the file:
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@@
     (thickness 1.6)
     (drawings 39)
-    (tracks 401)
+    (tracks 398)
     (zones 0)
     (modules 27)
@@
   (segment (start 104.300676 104.975169) (end 102.274831 104.975169) (width 0.6) (layer B.Cu) (net 1))
   (via (at 107.4 98.8) (size 0.8) (drill 0.4) (layers F.Cu B.Cu) (net 1))
-  (segment (start 107.502001 98.697999) (end 107.4 98.8) (width 0.6) (layer F.Cu) (net 1))
   (segment (start 108.087385 92.38) (end 108.44 92.38) (width 0.6) (layer B.Cu) (net 1))
   (segment (start 105.166248 95.301137) (end 108.087385 92.38) (width 0.6) (layer B.Cu) (net 1))
@@
   (segment (start 136.7 100) (end 139 100) (width 0.6) (layer B.Cu) (net 1))
   (segment (start 135.7 101) (end 136.7 100) (width 0.6) (layer B.Cu) (net 1))
-  (segment (start 107.60201 98.59799) (end 107.4 98.8) (width 0.6) (layer F.Cu) (net 1))
-  (segment (start 109.63549 98.59799) (end 107.60201 98.59799) (width 0.6) (layer F.Cu) (net 1))
   (segment (start 124.287177 100.912823) (end 122.4 102.8) (width 0.6) (layer B.Cu) (net 1))
   (segment (start 135.7 103.668602) (end 135.7 101) (width 0.6) (layer B.Cu) (net 1))
